File: Circuit/ESPlant-Sensors.sch (KiCad schematic (older format))
At the start: 6 parts, among them U301 BME280, U302 ADXL345

Commit message: ESP32 Version
Parts:
- removed C302: 1uF, FT:0603_CAP, symbol C
- removed U302: ADXL345, Plant:ADXL345, symbol ADXL345
- C301: footprint FT:0603_CAP -> Capacitors_SMD:C_0603_HandSoldering
- R301, R302: footprint FT:0603 -> Resistors_SMD:R_0603_HandSoldering
- U301: footprint Plant:BME280 -> libs:BME280
Connections:
- net labels removed: ADXL_INT
- wire segments 36 -> 18
- no-connect marks 1 -> 0
Other:
- note removed: "ADXL345 Fall Over Sensor / Accelerometer"
- note removed: "I2C Address 0x53\n"
Changed lines of the file:
@@
 EESchema Schematic File Version 2
-LIBS:ESPlant-rescue
-LIBS:freetronics_schematic
 LIBS:power
 LIBS:device
@@
 LIBS:valves
 LIBS:ESPlant
-LIBS:ESP8266
+LIBS:ESP32-footprints-Shem-Lib
+LIBS:freetronics_schematic
+LIBS:cp2102
+LIBS:relay
 LIBS:ESPlant-cache
 EELAYER 25 0
@@
 F 0 "U301" H 3400 3000 60  0000 C CNN
 F 1 "BME280" H 3150 3300 60  0000 C CNN
-F 2 "Plant:BME280" H 3150 3200 24  0000 C CNN
+F 2 "libs:BME280" H 3150 3200 24  0000 C CNN
 F 3 "" H 3150 3300 60  0000 C CNN
 	1    3150 3300
@@
 	1850 3450 2550 3450
 Wire Wire Line
-	2550 3550 1850 3550
+	1850 3550 2550 3550
 Text HLabel 1850 3550 0    60   Input ~ 0
 I2C_SCL
@@
 F 0 "R302" V 2330 3050 50  0000 C CNN
 F 1 "4.7K" V 2250 3050 50  0000 C CNN
-F 2 "FT:0603" V 2350 2850 24  0000 C CNN
+F 2 "Resistors_SMD:R_0603_HandSoldering" V 2350 2850 24  0000 C CNN
 F 3 "" H 2250 3050 60  0000 C CNN
 	1    2250 3050
@@
 F 0 "R301" V 2130 2950 50  0000 C CNN
 F 1 "4.7K" V 2050 2950 50  0000 C CNN
-F 2 "FT:0603" V 2150 2750 24  0000 C CNN
+F 2 "Resistors_SMD:R_0603_HandSoldering" V 2150 2750 24  0000 C CNN
 F 3 "" H 2050 2950 60  0000 C CNN
 	1    2050 2950
@@
 $EndComp
 Wire Wire Line
-	2250 2800 2250 2500
+	2250 2900 2250 2500
 Wire Wire Line
-	2050 2700 2050 2500
+	2050 2800 2050 2500
 Connection ~ 2250 2500
 Wire Wire Line
-	2250 3300 2250 3550
+	2250 3200 2250 3550
 Connection ~ 2250 3550
 Wire Wire Line
-	2050 3200 2050 3450
+	2050 3100 2050 3450
 Connection ~ 2050 3450
 Connection ~ 3250 2500
 $Comp
-L +3.3V #PWR043
+L +3.3V #PWR045
 U 1 1 564CDC53
 P 3250 2350
-F 0 "#PWR043" H 3250 2200 50  0001 C CNN
+F 0 "#PWR045" H 3250 2200 50  0001 C CNN
 F 1 "+3.3V" H 3250 2490 50  0000 C CNN
 F 2 "" H 3250 2350 60  0000 C CNN
@@
 $EndComp
 $Comp
-L GND #PWR044
+L GND #PWR046
 U 1 1 564CDC6D
 P 3250 4000
-F 0 "#PWR044" H 3250 3750 50  0001 C CNN
+F 0 "#PWR046" H 3250 3750 50  0001 C CNN
 F 1 "GND" H 3250 3850 50  0000 C CNN
 F 2 "" H 3250 4000 60  0000 C CNN
@@
 $EndComp
 Wire Wire Line
-	3250 4000 3250 3850
+	3250 3850 3250 4000
 Wire Wire Line
 	3250 3950 3100 3950
@@
 BME280 Temp/Humidity/Pressure\n
 $Comp
-L ADXL345 U302
-U 1 1 564CE29B
-P 6150 3100
-F 0 "U302" H 5600 2550 60  0000 C CNN
-F 1 "ADXL345" H 6150 2850 60  0000 C CNN
-F 2 "Plant:ADXL345" H 6100 2800 24  0000 C CNN
-F 3 "" H 6100 2800 60  0000 C CNN
-	1    6150 3100
-	1    0    0    -1
-$EndComp
-Text HLabel 4900 3250 0    60   Input ~ 0
-I2C_SDA
-Text HLabel 4900 3350 0    60   Input ~ 0
-I2C_SCL
-Wire Wire Line
-	4900 3250 5300 3250
-Wire Wire Line
-	4900 3350 5300 3350
-Wire Wire Line
-	5300 2950 5100 2950
-Wire Wire Line
-	5100 2950 5100 2300
-Wire Wire Line
-	4750 2300 6150 2300
-Wire Wire Line
-	5950 2300 5950 2450
-Wire Wire Line
-	6150 2200 6150 2450
-Connection ~ 5950 2300
-$Comp
-L +3.3V #PWR045
-U 1 1 564CE661
-P 6150 2200
-F 0 "#PWR045" H 6150 2050 50  0001 C CNN
-F 1 "+3.3V" H 6150 2340 50  0000 C CNN
-F 2 "" H 6150 2200 60  0000 C CNN
-F 3 "" H 6150 2200 60  0000 C CNN
-	1    6150 2200
-	1    0    0    -1
-$EndComp
-Connection ~ 6150 2300
-$Comp
-L GND #PWR046
-U 1 1 564CE6B9
-P 6150 4100
-F 0 "#PWR046" H 6150 3850 50  0001 C CNN
-F 1 "GND" H 6150 3950 50  0000 C CNN
-F 2 "" H 6150 4100 60  0000 C CNN
-F 3 "" H 6150 4100 60  0000 C CNN
-	1    6150 4100
-	1    0    0    -1
-$EndComp
-Wire Wire Line
-	6300 4000 6300 3900
-Wire Wire Line
-	6000 4000 6300 4000
-Wire Wire Line
-	6000 4000 6000 3900
-Wire Wire Line
-	6150 3900 6150 4100
-Connection ~ 6150 4000
-Wire Wire Line
-	6900 2950 7100 2950
-NoConn ~ 7100 2950
-$Comp
-L C C302
-U 1 1 564CEBB9
-P 4750 2650
-F 0 "C302" H 4775 2750 50  0000 L CNN
-F 1 "1uF" H 4550 2550 50  0000 L CNN
-F 2 "FT:0603_CAP" H 4600 2500 24  0000 C CNN
-F 3 "" H 4750 2650 60  0000 C CNN
-	1    4750 2650
-	1    0    0    -1
-$EndComp
-Wire Wire Line
-	4750 2800 4750 2950
-$Comp
-L GND #PWR047
-U 1 1 564CEC16
-P 4750 2950
-F 0 "#PWR047" H 4750 2700 50  0001 C CNN
-F 1 "GND" H 4750 2800 50  0000 C CNN
-F 2 "" H 4750 2950 60  0000 C CNN
-F 3 "" H 4750 2950 60  0000 C CNN
-	1    4750 2950
-	1    0    0    -1
-$EndComp
-Wire Wire Line
-	4750 2500 4750 2300
-Connection ~ 5100 2300
-$Comp
 L C C301
 U 1 1 564CEC68
@@
 F 0 "C301" H 3825 2800 50  0000 L CNN
 F 1 "1uF" H 3825 2600 50  0000 L CNN
-F 2 "FT:0603_CAP" H 3900 2550 24  0000 C CNN
+F 2 "Capacitors_SMD:C_0603_HandSoldering" H 3900 2550 24  0000 C CNN
 F 3 "" H 3800 2700 60  0000 C CNN
 	1    3800 2700
@@
 	3800 2850 3800 2950
 $Comp
-L GND #PWR048
+L GND #PWR047
 U 1 1 564CED66
 P 3800 2950
-F 0 "#PWR048" H 3800 2700 50  0001 C CNN
+F 0 "#PWR047" H 3800 2700 50  0001 C CNN
 F 1 "GND" H 3800 2800 50  0000 C CNN
 F 2 "" H 3800 2950 60  0000 C CNN
@@
 $EndComp
 Wire Wire Line
-	5300 3150 5000 3150
-Text Notes 4700 3900 0    60   ~ 0
-I2C Address 0x53\n
-Text Notes 4650 1750 0    79   ~ 0
-ADXL345 Fall Over Sensor / Accelerometer
-Wire Wire Line
-	6900 2850 7100 2850
-Text HLabel 7100 2850 2    60   Input ~ 0
-ADXL_INT
-Wire Wire Line
 	2400 3150 2400 2500
 Connection ~ 2400 2500
-Wire Wire Line
-	5000 3150 5000 2900
-Wire Wire Line
-	5000 2900 4750 2900
-Connection ~ 4750 2900
 $EndSCHEMATC
