File: Circuit/Power.sch (KiCad schematic (older format))
At the start: 19 parts, among them Q201 FDN340P, Q202 FDN340P, Q203 FDN340P, U201 CN3063, U202 MCP6002

Commit message: ESP32 Version
Parts:
- removed LED201: LED_GREEN, FT:LED-0805, symbol LED
- C201, C204: footprint FT:1210_CAP -> Capacitors_SMD:C_0805_HandSoldering
- C202: footprint FT:0603_CAP -> Capacitors_SMD:C_0603_HandSoldering
- C203: footprint FT:1210_CAP -> Capacitors_SMD:C_1210_HandSoldering
- D201: footprint FT:DIODE_SMA -> freetronics_footprints:DIODE_SMA
- LED202: value LED_RED -> CHG; footprint FT:LED-0805 -> LEDs:LED_0603
- Q201, Q202, Q203: footprint FT:SOT23_FET -> freetronics_footprints:SOT23_FET
- R201, R202, R203, R205, R206: footprint FT:0603 -> Resistors_SMD:R_0603_HandSoldering
- R204: value 7.15K 1% -> 3.6K 1%; footprint FT:0603 -> Resistors_SMD:R_0603_HandSoldering
- TH201: footprint FT:0603 -> Capacitors_SMD:C_0603_HandSoldering
- U201: footprint Plant:CN3063_SOIC8_EP -> libs:CN3063_SOIC8_EP
- U202: footprint FT:SO08_4mm -> freetronics_footprints:SO08_4mm
Connections:
- net labels removed: ~DONE
- wire segments 61 -> 56
- no-connect marks 0 -> 1
Other:
- moved on the sheet: LED202
