File: Circuit/ESPlant.kicad_pcb (KiCad board)
At the start: 2 copper layers, 97 x 77.5 mm, 77 parts, among them P1 SOIL, P101 CONN_DIGITAL, P102 CONN_ANALOG, P103 CONN_SERIAL, P104 CONN_I2C, P105 SOLAR, P106 USB_5PIN_SHELL, P109 CONN_PWR, P110 CONN_01X05, P111 UV, P112 TEMP, P113 NEOPIXEL, P114 PIR, Q101 FDN340P, Q201 FDN340P, Q202 FDN340P, Q203 FDN340P, SW101 RESET, SW102 PRGM, SW103 RESET, SW104 SS12D00, U101 STM32F042F, U103 ESP-12E, U201 CN3063, U202 MCP6002, U301 BME280, U302 ADXL345

Commit message: ESP32 Version
Parts:
- removed 1pin (x2): VAL**, Connect:1pin
- removed C102: 100nF, FT:0603_CAP
- removed C103: 10uF 16V, FT:1210_CAP
- removed C104: 100nF, FT:0603
- removed C302: 1uF, FT:0603_CAP
- removed G***: LOGO, Plant:lca2016_logo
- removed LED201: LED_GREEN, FT:LED-0805
- removed P101: CONN_DIGITAL, FT:1X08
- removed P102: CONN_ANALOG, FT:1X06
- removed P103: CONN_SERIAL, FT:1X02
- removed P104: CONN_I2C, FT:1X02
- removed P109: CONN_PWR, FT:1X03
- removed P110: CONN_01X05, FT:1X05
- removed P111: UV, FT:SCREWTERMINAL-3.5MM-3
- removed P112: TEMP, FT:SCREWTERMINAL-3.5MM-3
- removed P113: NEOPIXEL, FT:SCREWTERMINAL-3.5MM-3
- removed P114: PIR, FT:SCREWTERMINAL-3.5MM-3
- removed R101, R112: 1K, FT:0603
- removed R103, R108: 100K 1%, FT:0603
- removed R105, R109, R111, R113, R114: 10K, FT:0603
- removed R107: 121K 1%, FT:0603
- removed R110: 4.7K DNP, FT:0603
- removed SW103: RESET, FT:SW_PUSHBUTTON_PTH
- removed U101: STM32F042F, Plant:TSSOP20_4mm
- removed U103: ESP-12E, ESP:ESP-12E
- removed U302: ADXL345, Plant:ADXL345
- added C1: 10uF, Capacitors_SMD:C_0805_HandSoldering, F.Cu at (158.8, 83.4)
- added C2: 0.1uF, Capacitors_SMD:C_0603_HandSoldering, F.Cu at (158.8, 81.6)
- added C3: 10uF, Capacitors_SMD:C_0805_HandSoldering, F.Cu at (157.4, 88.4)
- added C4: 0.1uF, Capacitors_SMD:C_0603_HandSoldering, F.Cu at (155.6, 88.3)
- added C5: 1uF, Capacitors_SMD:C_0603_HandSoldering, F.Cu at (225.6, 83.1)
- added C6: 1uF, Capacitors_SMD:C_0603_HandSoldering, F.Cu at (225.1, 97.5)
- added D3: SS14, freetronics_footprints:DIODE_SMA, F.Cu at (217.5, 113.2)
- added D4: LED, LEDs:LED_0603, F.Cu at (213.4, 114.6)
- added P10: SOIL3, freetronics_footprints:SCREWTERMINAL-3.5MM-2, F.Cu at (146.0, 102.0)
- added P11: SOIL4, freetronics_footprints:SCREWTERMINAL-3.5MM-2, F.Cu at (146.0, 110.1)
- added P12: CONN_01X14, Pin_Headers:Pin_Header_Straight_1x14_Pitch2.54mm, F.Cu at (215.7, 62.3)
- added P2: IO17, freetronics_footprints:SCREWTERMINAL-3.5MM-3, F.Cu at (234.9, 107.4)
- added P3: IO18, freetronics_footprints:SCREWTERMINAL-3.5MM-3, F.Cu at (234.9, 95.0)
- added P4: CONN_01X14, Pin_Headers:Pin_Header_Straight_1x14_Pitch2.54mm, F.Cu at (181.9, 62.2)
- added P5: IO19, freetronics_footprints:SCREWTERMINAL-3.5MM-3, F.Cu at (234.9, 82.5)
- added P6: SOIL1, freetronics_footprints:SCREWTERMINAL-3.5MM-2, F.Cu at (146.0, 86.2)
- added P7: RELAY, freetronics_footprints:SCREWTERMINAL-3.5MM-3, F.Cu at (235.0, 124.8)
- added P8: SOIL2, freetronics_footprints:SCREWTERMINAL-3.5MM-2, F.Cu at (146.0, 94.1)
- added P9: CONN_01X10, Pin_Headers:Pin_Header_Straight_1x10_Pitch2.54mm, F.Cu at (210.2, 95.1)
- added Q1: S8050, TO_SOT_Packages_SMD:SOT-23_Handsoldering, F.Cu at (174.2, 76.3)
- added Q2: S8050, TO_SOT_Packages_SMD:SOT-23_Handsoldering, F.Cu at (173.7, 92.7)
- added Q3: 2N7002, TO_SOT_Packages_SMD:SOT-23_Handsoldering, F.Cu at (217.3, 107.2)
- added R1: 12K, Resistors_SMD:R_0603_HandSoldering, F.Cu at (171.2, 79.6)
- added R10: 470R, Resistors_SMD:R_0603_HandSoldering, F.Cu at (220.8, 97.5)
- added R2: 12K, Resistors_SMD:R_0603_HandSoldering, F.Cu at (177.2, 88.6)
- added R3: 470R, Resistors_SMD:R_0603_HandSoldering, F.Cu at (177.3, 82.4)
- added R4: 1K, Resistors_SMD:R_0603_HandSoldering, F.Cu at (218.0, 102.0)
- added R5: 1K, Resistors_SMD:R_0603_HandSoldering, F.Cu at (213.4, 110.7)
- added R6: 100K, Resistors_SMD:R_0603_HandSoldering, F.Cu at (151.6, 91.5)
- added R7: 100K, Resistors_SMD:R_0603_HandSoldering, F.Cu at (151.6, 96.5)
- added R8: 470R, Resistors_SMD:R_0603_HandSoldering, F.Cu at (221.2, 83.0)
- added R9: 100K, Resistors_SMD:R_0603_HandSoldering, F.Cu at (151.7, 112.1)
- added U1: CP2102, Housings_DFN_QFN:QFN-28-1EP_5x5mm_Pitch0.5mm, F.Cu at (162.8, 87.8)
- added U2: Relay, libs:SPDT_Songle_Relay, F.Cu at (219.8, 124.8)
- added U3: ESP32-WROOM, ESP32-footprints-Lib:ESP32-WROOM, F.Cu at (198.8, 73.8)
- C101, C107: footprint FT:0603_CAP -> Capacitors_SMD:C_0603_HandSoldering
- C106: value 100uF 16V X5R -> 100uF; footprint FT:1210_CAP -> Capacitors_SMD:C_1210_HandSoldering
- C201, C204: value 10uF 16V -> 10uF; footprint FT:1210_CAP -> Capacitors_SMD:C_0805_HandSoldering
- C202: value 100nF 16V -> 100nF; footprint FT:0603_CAP -> Capacitors_SMD:C_0603_HandSoldering
- C203: footprint FT:1210_CAP -> Capacitors_SMD:C_1210_HandSoldering
- D101: footprint FT:DIODE_SMA -> freetronics_footprints:DIODE_SMA
- F101: footprint FT:1210 -> freetronics_footprints:1210
- LED202: value LED_RED -> CHG; footprint FT:LED-0805 -> LEDs:LED_0603
- P1: value SOIL -> I2C; footprint FT:SCREWTERMINAL-3.5MM-3 -> Pin_Headers:Pin_Header_Straight_1x04_Pitch2.54mm
- P105: footprint FT:SCREWTERMINAL-3.5MM-2 -> freetronics_footprints:SCREWTERMINAL-3.5MM-2
- Q101, Q202, Q203: footprint FT:SOT23_FET -> freetronics_footprints:SOT23_FET
- R102: value 100K 1% -> 100K; footprint FT:0603 -> Resistors_SMD:R_0603_HandSoldering
- R104, R106, R202, R203, R206, R301, R302: footprint FT:0603 -> Resistors_SMD:R_0603_HandSoldering
- R204: value 7.15K 1% -> 3.6K; footprint FT:0603 -> Resistors_SMD:R_0603_HandSoldering
- R205: value 7.15K 1% -> 7.15K; footprint FT:0603 -> Resistors_SMD:R_0603_HandSoldering
- REG101: footprint FT:SOT23-5 -> freetronics_footprints:SOT23-5
- SW101, SW102: footprint FT:SW_PUSHBUTTON_PTH -> freetronics_footprints:SW_PUSHBUTTON_PTH
- SW104: value SS12D00 -> ON|OFF; footprint Plant:SS12D00 -> libs:SS12D00
- U201: footprint Plant:CN3063_SOIC8_EP -> libs:CN3063_SOIC8_EP
- U202: footprint FT:SO08_4mm -> freetronics_footprints:SO08_4mm
- moved P1 88.0 mm to (222.1, 62.3), turned to 90 degrees
- moved F101 74.5 mm to (168.6, 113.0), turned to 90 degrees
- moved SW101 70.6 mm to (223.3, 77.7), turned to 0 degrees
- moved SW102 70.0 mm to (223.0, 92.2), turned to 0 degrees
- moved D101 67.0 mm to (165.3, 113.1)
- moved R106 65.0 mm to (228.5, 107.3)
- moved Q101 64.6 mm to (224.0, 105.4)
- moved R104 64.4 mm to (228.4, 102.7)
- moved TH201 60.4 mm to (181.9, 128.1)
- moved BT101 60.3 mm to (181.9, 128.1), turned to 0 degrees
- moved SW104 58.3 mm to (167.8, 64.3), turned to 0 degrees
- moved C107 57.4 mm to (174.4, 66.2), turned to 90 degrees
- moved C301 55.6 mm to (232.5, 70.9)
- moved U301 55.6 mm to (236.5, 71.5)
- moved REG101 54.6 mm to (170.1, 70.8)
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Connections:
- net /GPIO14 renamed /IO16
- net /Power/USB_IN renamed /USB_VCC
- net /Power/VOUT renamed /VOUT
- P1 pad 1: /VCC_SENS -> GND
- P1 pad 2: /SOIL_2 -> /I2C_SCL
- P1 pad 3: /SOIL_1 -> /I2C_SDA
- P106 pad 4: (no net) -> Net-(P106-Pad4)
- R102 pad 1: /SOIL_1 -> /IO14
- R202 pad 2: Net-(LED201-PadA) -> Net-(LED202-Pad2)
- R301 pad 2: /I2C Sensors/I2C_SDA -> /I2C_SDA
- R302 pad 2: /I2C Sensors/I2C_SCL -> /I2C_SCL
- SW101 pad 2: /ESP_~RESET -> Net-(C5-Pad1)
- SW102 pad 2: /GPIO0_BOOT -> Net-(C6-Pad1)
- SW104 pad 3: (no net) -> Net-(SW104-Pad3)
- U201 pad 6: /Power/~DONE -> Net-(U201-Pad6)
- U301 pad 3: /I2C Sensors/I2C_SDA -> /I2C_SDA
- U301 pad 4: /I2C Sensors/I2C_SCL -> /I2C_SCL
Routing:
- net /I2C Sensors/I2C_SDA: track 136.5 -> 0.00 mm, vias 6 -> 0
- net /I2C Sensors/I2C_SCL: track 135.3 -> 0.00 mm, vias 7 -> 0
- net /ESP_~RESET: track 114.6 -> 0.00 mm, vias 2 -> 0
- net /IO16: track 144.8 -> 40.6 mm, vias 3 -> 0
- net /GPIO15: track 82.1 -> 0.00 mm, vias 3 -> 0
- net /GPIO0_BOOT: track 81.8 -> 0.00 mm, vias 2 -> 0
- net /SOIL1: track 0.00 -> 72.5 mm
- net /SOIL2: track 0.00 -> 66.1 mm
- net GND: track 204.5 -> 138.9 mm, vias 78 -> 26
- net /RXD: track 0.00 -> 65.6 mm, vias 0 -> 2
- net /GPIO12: track 64.8 -> 0.00 mm, vias 1 -> 0
- net /GPIO13: track 61.0 -> 0.00 mm, vias 3 -> 0
- net /EN: track 0.00 -> 58.7 mm, vias 0 -> 2
- net /IO12: track 0.00 -> 57.0 mm
- net /USB_D+: track 79.7 -> 23.2 mm, vias 0 -> 2
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- removed copper zone on F.Cu, net GND
Other:
- outline, holes or cut-outs redrawn
- board text added: "V2.0"
- board text added: "by John Spencer & Angus Gratton http://github.com/mage0r/ESPlant TAPR Open Hardware License"
- board text removed: "(GPIO0)"
- board text removed: "+"
- board text removed: "+3.3V"
- board text removed: "+VSen"
- board text removed: "-"
- board text removed: "ADC0"
- board text removed: "ADC1"
- board text removed: "ADC2"
- board text removed: "ADC3"
- board text removed: "ADC4"
- board text removed: "Charged"
- board text removed: "Charging"
- board text removed: "Designed for LCA2016 Open Hardware MiniConf by John Spencer & Angus Gratton http://github.com/mage0r/ESPlant TAPR Open Hardware License"
- board text removed: "ESP FLASH"
- board text removed: "ESP RESET"
- board text removed: "GND"
- board text removed: "GPIO0"
- board text removed: "GPIO12"
- board text removed: "GPIO13"
- board text removed: "GPIO14"
- board text removed: "GPIO15"
- board text removed: "GPIO2"
- board text removed: "LEDS"
- board text removed: "MAX 7V/1A"
- board text removed: "OFF"
- board text removed: "ON"
- board text removed: "PIR SENSOR"
- board text removed: "RX (GPIO3)"
- board text removed: "SCL"
- board text removed: "SCL/GPIO5"
- board text removed: "SDA"
- board text removed: "SDA/GPIO4"
- board text removed: "SOIL MOISTURE"
- board text removed: "SOLAR PANEL"
- board text removed: "STM DEBUG"
- board text removed: "STM RESET"
- board text removed: "SWCLK"
- board text removed: "SWDIO"
- board text removed: "TEMP SENSOR"
- board text removed: "TX (GPIO1)"
- board text removed: "UV SENSOR"
- board text removed: "V1.5"
- board text removed: "WS2812B"
- board text removed: "~RST"

Commit message: Updated pcb.
Completed a missing track.
Added some ground plane to the regulator.
Changed some silkscreen test.
Parts:
- moved R6 5.59 mm to (155.8, 95.1), turned to 0 degrees
- moved R9 4.52 mm to (156.2, 112.1)
- moved R203 4.28 mm to (199.8, 107.4), turned to 270 degrees
- moved Q202 3.96 mm to (195.7, 107.1)
- moved R7 2.46 mm to (152.7, 98.7), turned to 270 degrees
- moved R102 2.26 mm to (153.7, 104.6), turned to 270 degrees
- moved R104 2.05 mm to (226.5, 101.9)
- moved R301 1.68 mm to (227.3, 66.6)
- moved R106 1.54 mm to (227.4, 108.4)
Routing:
- net /IO0: track 19.0 -> 67.6 mm, vias 0 -> 2
- net /VOUT: track 108.4 -> 97.5 mm
- net /IO16: track 40.6 -> 43.7 mm
- net /Power/GIN: track 13.7 -> 16.5 mm
- net +3V3: track 198.2 -> 195.6 mm
- net GND: track 138.9 -> 140.2 mm, vias 26 -> 28
- net /I2C_SDA: track 46.9 -> 47.7 mm
Other:
- board text added: "+3v3"
- board text added: "GND"
- board text added: "IO17"
- board text added: "IO18"
- board text added: "IO19"
- board text added: "OFF|ON"
- board text added: "RELAY"
- board text added: "SCL"
- board text added: "SDA"
- board text added: "SOIL1"
- board text added: "SOIL2"
- board text added: "SOIL3"
- board text added: "SOIL4"

Commit message: Updates, I guess
Parts:
- moved D102 4.04 mm to (158.1, 69.9)
Routing:
- net /SOIL2: track 66.1 -> 73.7 mm
- net /Power/SOLAR_IN: track 11.2 -> 14.1 mm
- net GND: track 140.2 -> 142.6 mm, vias 28 -> 30
- net /SOIL1: track 72.2 -> 73.3 mm
- net +3V3: track 195.6 -> 196.7 mm
- net /IO14: track 55.5 -> 56.5 mm
Changed lines of the file:
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@@
   (general
     (links 212)
-    (no_connects 6)
+    (no_connects 0)
     (area 140.248029 58.531 239.075001 138.519)
     (thickness 1.6)
     (drawings 48)
-    (tracks 736)
+    (tracks 757)
     (zones 0)
     (modules 79)
@@
   )
   (setup
-    (last_trace_width 0.15)
+    (last_trace_width 0.6)
     (user_trace_width 0.15)
     (user_trace_width 0.2)
@@
   )
   (module FT:DIODE_SMA (layer F.Cu)
-    (at 154.22 68.66 180)
+    (at 158.07 69.89 180)
     (attr smd)
-    (fp_text reference D102 (at 2.45 2.19 180) (layer F.SilkS)
+    (fp_text reference D102 (at -1.22 2.08 180) (layer F.SilkS)
       (effects (font (size 0.7 0.7) (thickness 0.15)))
     )
@@
     (tags "capacitor 0805")
     (attr smd)
-    (fp_text reference C3 (at 3.79 -0.06 270) (layer F.SilkS)
+    (fp_text reference C3 (at 3.2 -0.01 270) (layer F.SilkS)
       (effects (font (size 1 1) (thickness 0.15)))
     )
@@
       (effects (font (size 1 1) (thickness 0.15)))
     )
-    (fp_text user %R (at 3.79 -0.06 270) (layer F.Fab)
+    (fp_text user %R (at 3.18 -0.01 270) (layer F.Fab)
       (effects (font (size 1 1) (thickness 0.15)))
     )
@@
     (tags "capacitor 0603")
     (attr smd)
-    (fp_text reference C4 (at 3.82 0.02 270) (layer F.SilkS)
+    (fp_text reference C4 (at 3.3 0.07 270) (layer F.SilkS)
       (effects (font (size 1 1) (thickness 0.15)))
     )
@@
       (effects (font (size 1 1) (thickness 0.15)))
     )
-    (fp_text user %R (at 3.81 0.01 270) (layer F.Fab)
+    (fp_text user %R (at 3.3 0.05 270) (layer F.Fab)
       (effects (font (size 1 1) (thickness 0.15)))
     )
@@
     (tags "resistor 0603")
     (attr smd)
-    (fp_text reference R2 (at 0 -1.45 90) (layer F.SilkS)
+    (fp_text reference R2 (at 0 1.47 90) (layer F.SilkS)
       (effects (font (size 1 1) (thickness 0.15)))
     )
-    (fp_text value 12K (at 0 1.55 90) (layer F.Fab)
+    (fp_text value 12K (at 0.02 -1.4 90) (layer F.Fab)
       (effects (font (size 1 1) (thickness 0.15)))
     )
-    (fp_text user %R (at 0 -1.45 90) (layer F.Fab)
+    (fp_text user %R (at 0 -1.45 90) (layer F.Fab) hide
       (effects (font (size 1 1) (thickness 0.15)))
     )
@@
     (tags "resistor 0603")
     (attr smd)
-    (fp_text reference R9 (at 0 -1.45 90) (layer F.SilkS)
+    (fp_text reference R9 (at -0.02 1.45 90) (layer F.SilkS)
       (effects (font (size 1 1) (thickness 0.15)))
     )
-    (fp_text value 100K (at 0 1.55 90) (layer F.Fab)
+    (fp_text value 100K (at -2.66 0.03 180) (layer F.Fab)
       (effects (font (size 1 1) (thickness 0.15)))
     )
-    (fp_text user %R (at 0 -1.45 90) (layer F.Fab)
+    (fp_text user %R (at -0.02 1.45 90) (layer F.Fab)
       (effects (font (size 1 1) (thickness 0.15)))
     )
@@
   (segment (start 168.63 122.36) (end 166.06 124.93) (width 0.6) (layer F.Cu) (net 1))
   (segment (start 166.06 124.93) (end 162.89 128.1) (width 0.6) (layer F.Cu) (net 1))
+  (segment (start 160.21884 69.89) (end 161.42 69.89) (width 0.6) (layer F.Cu) (net 2))
+  (segment (start 161.45 69.92) (end 161.44 69.91) (width 0.6) (layer B.Cu) (net 2))
+  (via (at 161.45 69.92) (size 0.6) (drill 0.3) (layers F.Cu B.Cu) (net 2))
+  (segment (start 161.42 69.89) (end 161.45 69.92) (width 0.6) (layer F.Cu) (net 2))
+  (segment (start 156.94 95.14) (end 158.18 95.14) (width 0.6) (layer F.Cu) (net 2))
+  (via (at 158.18 95.14) (size 0.6) (drill 0.3) (layers F.Cu B.Cu) (net 2))
+  (segment (start 152.71 99.79) (end 151.69 99.79) (width 0.6) (layer F.Cu) (net 2))
+  (via (at 151.68 99.8) (size 0.6) (drill 0.3) (layers F.Cu B.Cu) (net 2))
+  (segment (start 151.69 99.79) (end 151.68 99.8) (width 0.6) (layer F.Cu) (net 2))
   (via (at 170.17 70.7815) (size 0.6) (drill 0.3) (layers F.Cu B.Cu) (net 2))
   (via (at 171.3985 70.7815) (size 0.6) (drill 0.3) (layers F.Cu B.Cu) (net 2))
@@
   (segment (start 226.03 97.48) (end 227.2 97.48) (width 0.6) (layer F.Cu) (net 2))
   (via (at 227.2 97.48) (size 0.6) (drill 0.3) (layers F.Cu B.Cu) (net 2))
-  (segment (start 156.36884 68.66) (end 157.51 68.66) (width 0.6) (layer F.Cu) (net 2))
-  (via (at 157.51 68.66) (size 0.6) (drill 0.3) (layers F.Cu B.Cu) (net 2))
   (segment (start 206.13 106.07) (end 207.31 106.07) (width 0.6) (layer F.Cu) (net 2))
   (via (at 207.31 106.07) (size 0.6) (drill 0.3) (layers F.Cu B.Cu) (net 2))
@@
   (segment (start 168.55 76.45) (end 168.55 72.78798) (width 0.6) (layer F.Cu) (net 3))
   (segment (start 168.55 72.78798) (end 169.19004 72.14794) (width 0.6) (layer F.Cu) (net 3))
+  (segment (start 161.27 85.37) (end 161.27 84.57) (width 0.15) (layer F.Cu) (net 4))
+  (segment (start 161.27 84.57) (end 161.45 84.39) (width 0.15) (layer F.Cu) (net 4))
+  (segment (start 160.07 83.38) (end 161.41 83.38) (width 0.15) (layer F.Cu) (net 4))
+  (segment (start 161.41 83.38) (end 161.45 83.34) (width 0.15) (layer F.Cu) (net 4))
   (segment (start 181.75 103.88) (end 209.87 103.88) (width 0.6) (layer F.Cu) (net 4))
   (segment (start 209.87 103.88) (end 212.01 101.74) (width 0.6) (layer F.Cu) (net 4))
@@
   (segment (start 159.72 81.61) (end 161.45 81.61) (width 0.6) (layer F.Cu) (net 4))
   (segment (start 161.45 84.39) (end 161.45 83.34) (width 0.6) (layer F.Cu) (net 4))
-  (segment (start 160.07 83.38) (end 161.42 83.38) (width 0.6) (layer F.Cu) (net 4))
-  (segment (start 161.42 83.38) (end 161.45 83.35) (width 0.6) (layer F.Cu) (net 4))
-  (segment (start 161.45 83.35) (end 161.45 83.34) (width 0.6) (layer F.Cu) (net 4))
-  (segment (start 161.77 85.37) (end 161.45 85.37) (width 0.2) (layer F.Cu) (net 4))
-  (segment (start 161.45 84.39) (end 161.45 84.814264) (width 0.6) (layer F.Cu) (net 4))
   (segment (start 161.45 84.814264) (end 161.45 85.37) (width 0.6) (layer F.Cu) (net 4))
+  (segment (start 161.45 84.39) (end 161.45 84.814264) (width 0.6) (layer F.Cu) (net 4))
+  (segment (start 161.77 85.37) (end 161.45 85.37) (width 0.2) (layer F.Cu) (net 4))
   (segment (start 171.08996 72.14794) (end 171.08996 73.28004) (width 0.6) (layer F.Cu) (net 4))
   (segment (start 171.08996 73.28004) (end 171.08 73.29) (width 0.6) (layer F.Cu) (net 4))
@@
   (segment (start 222.88018 105.38) (end 222.88018 110.07899) (width 0.6) (layer F.Cu) (net 8))
   (segment (start 217.59033 115.36884) (end 217.49 115.36884) (width 0.6) (layer F.Cu) (net 8))
+  (segment (start 153.7 71.37018) (end 154.44098 71.37018) (width 0.6) (layer F.Cu) (net 9))
+  (segment (start 154.44098 71.37018) (end 155.92116 69.89) (width 0.6) (layer F.Cu) (net 9))
   (segment (start 152.07116 68.66) (end 152.07116 69.74134) (width 0.6) (layer F.Cu) (net 9))
   (segment (start 152.07116 69.74134) (end 153.7 71.37018) (width 0.6) (layer F.Cu) (net 9))
@@
   (segment (start 189.8 71.07) (end 185.64 71.07) (width 0.6) (layer F.Cu) (net 29))
   (segment (start 185.64 71.07) (end 181.88 67.31) (width 0.6) (layer F.Cu) (net 29))
+  (segment (start 154.23 94.2) (end 154.23 94.63) (width 0.15) (layer F.Cu) (net 30))
+  (segment (start 154.23 94.63) (end 154.74 95.14) (width 0.15) (layer F.Cu) (net 30))
   (segment (start 146 89.68758) (end 151.49758 89.68758) (width 0.15) (layer F.Cu) (net 30))
   (segment (start 151.49758 89.68758) (end 154.23 92.42) (width 0.15) (layer F.Cu) (net 30))
-  (segment (start 154.23 92.42) (end 154.23 95.7) (width 0.15) (layer F.Cu) (net 30))
+  (segment (start 154.23 92.42) (end 154.23 94.2) (width 0.15) (layer F.Cu) (net 30))
+  (segment (start 154.23 94.2) (end 154.23 95.7) (width 0.15) (layer F.Cu) (net 30))
   (segment (start 154.23 95.7) (end 154.83 96.3) (width 0.15) (layer F.Cu) (net 30))
   (segment (start 154.83 96.3) (end 175.47 96.3) (width 0.15) (layer F.Cu) (net 30))
@@
   (segment (start 189.8 72.34) (end 184.37 72.34) (width 0.6) (layer F.Cu) (net 30))
   (segment (start 184.37 72.34) (end 181.88 69.85) (width 0.6) (layer F.Cu) (net 30))
+  (segment (start 152.71 97.59) (end 146.01758 97.59) (width 0.15) (layer F.Cu) (net 31))
+  (segment (start 146.01758 97.59) (end 146 97.60758) (width 0.15) (layer F.Cu) (net 31))
+  (segment (start 152.71 97.59) (end 152.28516 97.59) (width 0.15) (layer F.Cu) (net 31))
+  (segment (start 152.28516 97.59) (end 152.26758 97.60758) (width 0.15) (layer F.Cu) (net 31))
+  (segment (start 152.26758 97.60758) (end 152.71 97.59) (width 0.15) (layer F.Cu) (net 31))
   (segment (start 180.02 93.43) (end 175.84242 97.60758) (width 0.15) (layer F.Cu) (net 31))
   (segment (start 175.84242 97.60758) (end 173.62242 97.60758) (width 0.15) (layer F.Cu) (net 31))
@@
   (segment (start 186.209991 84.240009) (end 187.95 82.5) (width 0.6) (layer F.Cu) (net 38))
   (segment (start 187.95 82.5) (end 189.8 82.5) (width 0.6) (layer F.Cu) (net 38))
+  (segment (start 153.89 102.54) (end 153.89 103.26) (width 0.15) (layer F.Cu) (net 39))
+  (segment (start 153.89 103.26) (end 153.69 103.46) (width 0.15) (layer F.Cu) (net 39))
   (segment (start 146 105.54758) (end 150.92242 105.54758) (width 0.15) (layer F.Cu) (net 39))
   (segment (start 174.67 99.92) (end 181.88 92.71) (width 0.15) (layer F.Cu) (net 39))
   (segment (start 154.78 99.92) (end 174.67 99.92) (width 0.15) (layer F.Cu) (net 39))
   (segment (start 153.89 100.81) (end 154.78 99.92) (width 0.15) (layer F.Cu) (net 39))
-  (segment (start 153.89 102.58) (end 153.89 100.81) (width 0.15) (layer F.Cu) (net 39))
+  (segment (start 153.89 102.58) (end 153.89 102.54) (width 0.15) (layer F.Cu) (net 39))
+  (segment (start 153.89 102.54) (end 153.89 100.81) (width 0.15) (layer F.Cu) (net 39))
   (segment (start 150.92242 105.54758) (end 153.89 102.58) (width 0.15) (layer F.Cu) (net 39))
   (segment (start 186.96 87.63) (end 186.96 84.76) (width 0.6) (layer F.Cu) (net 39))
