File: Circuit/ESPlant.sch (KiCad schematic (older format))
At the start: 49 parts, among them P1 SOIL, P101 CONN_DIGITAL, P102 CONN_ANALOG, P103 CONN_SERIAL, P104 CONN_I2C, P105 SOLAR, P106 USB_5PIN_SHELL, P109 CONN_PWR, P110 CONN_01X05, P111 UV, P112 TEMP, P113 NEOPIXEL, P114 PIR, Q101 FDN340P, SW101 RESET, SW102 PRGM, SW103 RESET, SW104 SS12D00, U101 STM32F042F, U103 ESP-12E

Commit message: ESP32 Version
Parts:
- removed C102, C104: 100nF, FT:0603_CAP, symbol C
- removed C103: 10uF 16V, FT:1210_CAP, symbol C
- removed MH101, MH102, MH103, MH104: TEST_1P, Connect:1pin, symbol TEST_1P
- removed P1: SOIL, FT:SCREWTERMINAL-3.5MM-3, symbol CONN_01X03
- removed P101: CONN_DIGITAL, FT:1X08, symbol CONN_01X08
- removed P102: CONN_ANALOG, FT:1X06, symbol CONN_01X06
- removed P103: CONN_SERIAL, FT:1X02, symbol CONN_01X02
- removed P104: CONN_I2C, FT:1X02, symbol CONN_01X02
- removed P109: CONN_PWR, FT:1X03, symbol CONN_01X03
- removed P110: CONN_01X05, FT:1X05, symbol CONN_01X05
- removed P111: UV, FT:SCREWTERMINAL-3.5MM-3, symbol CONN_01X03
- removed P112: TEMP, FT:SCREWTERMINAL-3.5MM-3, symbol CONN_01X03
- removed P113: NEOPIXEL, FT:SCREWTERMINAL-3.5MM-3, symbol CONN_01X03
- removed P114: PIR, FT:SCREWTERMINAL-3.5MM-3, symbol CONN_01X03
- removed R101, R112: 1K, FT:0603, symbol R
- removed R103, R108: 100K 1%, FT:0603, symbol R
- removed R105, R109, R113, R114: 10K, FT:0603, symbol R
- removed R107: 121K 1%, FT:0603, symbol R
- removed R110: 4.7K DNP, FT:0603, symbol R
- removed SW103: RESET, FT:SW_PUSHBUTTON_PTH, symbol SW_PUSH
- removed U101: STM32F042F, Plant:TSSOP20_4mm, symbol STM32F042F
- removed U103: ESP-12E, ESP:ESP-12E, symbol ESP-12E
- added C1, C3: 10uF, Capacitors_SMD:C_0805_HandSoldering, symbol C
- added C2, C4: 0.1uF, Capacitors_SMD:C_0603_HandSoldering, symbol C
- added C5, C6: 1uF, Capacitors_SMD:C_0603_HandSoldering, symbol C
- added D1, D2: ESD05V88D-LC, libs:SOD-882, symbol TVS
- added D3: SS14, freetronics_footprints:DIODE_SMA, symbol DIODE_SCHOTTKY
- added D4: LED, LEDs:LED_0603, symbol LED
- added P1: I2C, Pin_Headers:Pin_Header_Straight_1x04_Pitch2.54mm, symbol CONN_01X04
- added P10: SOIL3, freetronics_footprints:SCREWTERMINAL-3.5MM-2, symbol CONN_01X02
- added P11: SOIL4, freetronics_footprints:SCREWTERMINAL-3.5MM-2, symbol CONN_01X02
- added P12, P4: CONN_01X14, Pin_Headers:Pin_Header_Straight_1x14_Pitch2.54mm, symbol CONN_01X14
- added P2: IO17, freetronics_footprints:SCREWTERMINAL-3.5MM-3, symbol CONN_01X03
- added P3: IO18, freetronics_footprints:SCREWTERMINAL-3.5MM-3, symbol CONN_01X03
- added P5: IO19, freetronics_footprints:SCREWTERMINAL-3.5MM-3, symbol CONN_01X03
- added P6: SOIL1, freetronics_footprints:SCREWTERMINAL-3.5MM-2, symbol CONN_01X02
- added P7: RELAY, freetronics_footprints:SCREWTERMINAL-3.5MM-3, symbol CONN_01X03
- added P8: SOIL2, freetronics_footprints:SCREWTERMINAL-3.5MM-2, symbol CONN_01X02
- added P9: CONN_01X10, Pin_Headers:Pin_Header_Straight_1x10_Pitch2.54mm, symbol CONN_01X10
- added Q1, Q2: S8050, TO_SOT_Packages_SMD:SOT-23_Handsoldering, symbol Q_NPN_BEC
- added Q3: 2N7002, TO_SOT_Packages_SMD:SOT-23_Handsoldering, symbol 2N7002
- added R1, R2: 12K, Resistors_SMD:R_0603_HandSoldering, symbol R
- added R10, R3: 470R, Resistors_SMD:R_0603_HandSoldering, symbol R
- added R4, R5: 1K, Resistors_SMD:R_0603_HandSoldering, symbol R
- added R6, R7, R9: 100K 1%, Resistors_SMD:R_0603_HandSoldering, symbol R
- added U1: CP2102, Housings_DFN_QFN:QFN-28-1EP_5x5mm_Pitch0.5mm, symbol CP2102
- added U2: Relay, libs:SPDT_Songle_Relay, symbol Relay
- added U3: ESP32-WROOM, ESP32-footprints-Lib:ESP32-WROOM, symbol ESP32-WROOM
- BT101: footprint Plant:CR123_Holder -> libs:CR123_Holder
- C101, C107: footprint FT:0603_CAP -> Capacitors_SMD:C_0603_HandSoldering
- C106: footprint FT:1210_CAP -> Capacitors_SMD:C_1210_HandSoldering
- D101, D102: footprint FT:DIODE_SMA -> freetronics_footprints:DIODE_SMA
- F101: footprint FT:1210 -> freetronics_footprints:1210
- P105: footprint FT:SCREWTERMINAL-3.5MM-2 -> freetronics_footprints:SCREWTERMINAL-3.5MM-2
- P106: footprint FT:USB-MICRO-5pin_PTHMOUNT -> freetronics_footprints:USB-MICRO-5pin_PTHMOUNT
- Q101: footprint FT:SOT23_FET -> freetronics_footprints:SOT23_FET
- R102, R104, R106: footprint FT:0603 -> Resistors_SMD:R_0603_HandSoldering
- R8: renamed from R111; value 10K -> 470R; footprint FT:0603 -> Resistors_SMD:R_0603_HandSoldering
- REG101: footprint FT:SOT23-5 -> freetronics_footprints:SOT23-5
- SW101, SW102: footprint FT:SW_PUSHBUTTON_PTH -> freetronics_footprints:SW_PUSHBUTTON_PTH
- SW104: value SS12D00 -> ON|OFF; footprint Plant:SS12D00 -> libs:SS12D00
Connections:
- net labels added: ACTIVE, CLK, CMD, CTS, DCD, DSR, DTR, EN, IO0, IO12, IO13, IO14, IO15, IO16, IO17, IO18, IO19, IO2, IO21, IO22, IO23, IO25, IO26, IO27, IO32, IO33, IO34, IO35, IO4, IO5, RI, RTS, RXD, SD0, SD1, SD2, SD3, SOIL1, SOIL2, SOIL3, SOIL4, Sensor_VN, Sensor_VP, TXD
- net labels removed: ADC0, ADC1, ADC2, ESP_EN, ESP_~RESET, GPIO0, GPIO0_BOOT, GPIO12, GPIO13, GPIO14, GPIO15, GPIO16, GPIO2, SOIL_1, SOIL_2, STM_RXD, STM_SWCLK, STM_SWDIO, STM_TXD, STM_~RESET
- wire segments 168 -> 210
- no-connect marks 13 -> 5
Other:
- note added: "Digital 1"
- note added: "Digital 2"
- note added: "Digital 3"
- note added: "Relay"
- note added: "VCC_Sense"
- note removed: "Breakouts\nfor External Connections"
- note removed: "Buttons & LEDs"
- note removed: "ESP Pin Strapping"
- note removed: "ESP8266 WiFi Microcontroller"
- note removed: "External Sensor Screw Terminals"
- note removed: "Input voltage\nmonitor via divider\n0-7V -> 0-3.2V,\n"
- note removed: "Mounting Holes\n"
- note removed: "STM32 SWD\nProgramming\nHeader (Optional)"
- note removed: "STM32 USB/Serial & ADC Combo"
- note removed: "Soil Moisture Sensors\n"
- note removed: "VCC_SENS is used to\npulse current through\nsoil moisture sensors."
- moved on the sheet: C106, C107, Q101, R102, R104, R106, R8, SW102

Commit message: Updates, I guess
Parts:
- added R?: 12K, Resistors_SMD:R_0603_HandSoldering, symbol R
Connections:
- net +3V3: now also R?.2
- net CLK: now also P9.6 (P6); no longer P9.5 (P5)
- net CMD: now also P9.5 (P5); no longer P9.6 (P6)
- net EN: now also R?.1
- net GND: now also P9.1 (P1); no longer P9.10 (P10)
- net IO13: now also P9.2 (P2); no longer P9.9 (P9)
- net IO15: now also P9.9 (P9); no longer P9.2 (P2)
- net IO2: now also P9.10 (P10); no longer P9.1 (P1)
- net SD0: now also P9.7 (P7); no longer P9.4 (P4)
- net SD1: now also P9.8 (P8); no longer P9.3 (P3)
- net SD2: now also P9.3 (P3); no longer P9.8 (P8)
- net SD3: now also P9.4 (P4); no longer P9.7 (P7)
Changed lines of the file:
@@
 F 3 "" H 9150 3500 50  0000 C CNN
 	1    9150 3500
-	0    1    1    0
+	0    -1   1    0
 $EndComp
 Connection ~ 8700 3000
@@
 Text Label 2750 6900 2    60   ~ 0
 USB_VCC
+$Comp
+L +3.3V #PWR?
+U 1 1 58FF9292
+P 10700 3450
+F 0 "#PWR?" H 10700 3300 50  0001 C CNN
+F 1 "+3.3V" H 10700 3590 50  0000 C CNN
+F 2 "" H 10700 3450 60  0000 C CNN
+F 3 "" H 10700 3450 60  0000 C CNN
+	1    10700 3450
+	1    0    0    -1
+$EndComp
+Text Label 10950 3800 2    60   ~ 0
+EN
+$Comp
+L R R?
+U 1 1 58FFA417
+P 10700 3600
+F 0 "R?" V 10780 3600 50  0000 C CNN
+F 1 "12K" V 10700 3600 50  0000 C CNN
+F 2 "Resistors_SMD:R_0603_HandSoldering" V 10630 3600 24  0000 C CNN
+F 3 "" H 10700 3600 30  0000 C CNN
+	1    10700 3600
+	-1   0    0    1
+$EndComp
+Wire Wire Line
+	10700 3750 10700 3800
+Wire Wire Line
+	10700 3800 10950 3800
 $EndSCHEMATC
